Commit message: bytta lidar_link til laser
Co-authored-by: Copilot <copilot@github.com>

File: src/ros_gz_description/models/xacro_test/test.urdf.xacro (robot description, xacro)
@@ -236,8 +236,8 @@
   <joint name="lidar_sensor_joint" type="fixed">
     <parent link="lidar_hinge_link"/>
-    <child link="lidar_link"/>
+    <child link="laser"/>
     <origin xyz="0 0 0.032" rpy="0 0 0"/> <!-- 32 mm opp (Z-aksen) -->
   </joint>
-  <link name="lidar_link">
+  <link name="laser">
     <visual>
       <origin xyz="0 0 0" rpy="0 0 0"/>
@@ -260,6 +260,6 @@
     </inertial>
   </link>
-  <!-- Gazebo sensor on lidar_link -->
-  <gazebo reference="lidar_link">
+  <!-- Gazebo sensor on laser -->
+  <gazebo reference="laser">
     <sensor name="lidar" type="gpu_lidar">
       <always_on>true</always_on>
@@ -267,5 +267,5 @@
       <visualize>true</visualize>
       <topic>/scan</topic>
-      <gz_frame_id>lidar_link</gz_frame_id>
+      <gz_frame_id>laser</gz_frame_id>
       <lidar>
         <scan>

Commit message: base_footprint
Co-authored-by: Copilot <copilot@github.com>

File: src/ros_gz_description/models/xacro_test/test.urdf.xacro (robot description, xacro)
@@ -72,7 +72,7 @@
                          via body_link)
        ============================================================ -->
-  <link name="base_link"/>
+  <link name="base_footprint"/>
   <joint name="body_link_joint" type="fixed">
-    <parent link="base_link"/>
+    <parent link="base_footprint"/>
     <child link="body_link"/>
   </joint>
