Commit message: Laget gregor leunch-fil. Lagt til kalmanfilter, og lidar sweep_node

File: src/ros_gz_description/models/xacro_test/test.urdf.xacro (robot description, xacro)
@@ -218,9 +218,24 @@
     </collision>
   </gazebo>
-  <!-- LiDAR link -->
-  <joint name="lidar_joint" type="fixed">
-    <parent link="body_link"/>
+  <!-- HINGE LINK (Vippepunktet) -->
+  <joint name="lidar_joint" type="revolute">
+    <parent link="body_link"/>
+    <child link="lidar_hinge_link"/>
+    <origin xyz="0 0 ${s1+s5}" rpy="0 0 0"/>
+    <axis xyz="0 1 0"/> <!-- Vipper opp og ned om Y-aksen -->
+    <limit lower="-0.785398" upper="0.785398" effort="10.0" velocity="5.0"/> <!-- +/- 45 grader -->
+    <dynamics damping="0.1" friction="0.1"/>
+  </joint>
+  <link name="lidar_hinge_link">
+    <inertial>
+      <mass value="0.05"/>
+      <inertia ixx="0.0001" ixy="0" ixz="0" iyy="0.0001" iyz="0" izz="0.0001"/>
+    </inertial>
+  </link>
+  <!-- SENSOR LINK (Forskyvningen på 32mm over vippepunktet) -->
+  <joint name="lidar_sensor_joint" type="fixed">
+    <parent link="lidar_hinge_link"/>
     <child link="lidar_link"/>
-    <origin xyz="0 0 ${s1+s5}" rpy="0 0 0"/>
+    <origin xyz="0 0 0.032" rpy="0 0 0"/> <!-- 32 mm opp (Z-aksen) -->
   </joint>
   <link name="lidar_link">
@@ -262,8 +277,8 @@
           </horizontal>
           <vertical>
-            <samples>16</samples>
+            <samples>1</samples>
             <resolution>1</resolution>
-            <min_angle>-0.10</min_angle>
-            <max_angle>0.10</max_angle>
+            <min_angle>0.0</min_angle>
+            <max_angle>0.0</max_angle>
           </vertical>
         </scan>
@@ -303,10 +318,10 @@
   <!-- Gazebo camera sensor -->
   <gazebo reference="camera_link">
-    <sensor name="front_thermal_camera" type="thermal_camera">
+    <sensor name="front_camera" type="camera">
       <always_on>true</always_on>
       <update_rate>20</update_rate>
       <visualize>true</visualize>
-      <topic>/camera/thermal/image_raw</topic>
-      <camera_info_topic>/camera/thermal/camera_info</camera_info_topic>
+      <topic>/camera/image_raw</topic>
+      <camera_info_topic>/camera/camera_info</camera_info_topic>
       <thermal_camera>
         <horizontal_fov>1.3962634</horizontal_fov>
@@ -392,5 +407,14 @@
     <!-- JointStatePublisher plugin -->
     <plugin filename="gz-sim-joint-state-publisher-system"
-            name="gz::sim::systems::JointStatePublisher"/>
+            name="gz::sim::systems::JointStatePublisher">
+    </plugin>
+    <!-- Lidar Pitch Controller -->
+    <plugin filename="gz-sim-joint-position-controller-system"
+            name="gz::sim::systems::JointPositionController">
+      <joint_name>lidar_joint</joint_name>
+      <p_gain>10.0</p_gain>
+      <i_gain>0.1</i_gain>
+      <d_gain>0.1</d_gain>
+    </plugin>
   </gazebo>
 </robot>

Commit message: prøver å snu imu i xacro

File: src/ros_gz_description/models/xacro_test/test.urdf.xacro (robot description, xacro)
@@ -345,5 +345,5 @@
     <parent link="body_link"/>
     <child link="imu_link"/>
-    <origin xyz="0.1 0 ${s1 + s5}" rpy="0 0 0"/>
+    <origin xyz="0.1 0 ${s1 + s5}" rpy="0 0 3.14159"/>
   </joint>
   <link name="imu_link">

Commit message: var ikke det

File: src/ros_gz_description/models/xacro_test/test.urdf.xacro (robot description, xacro)
@@ -345,5 +345,5 @@
     <parent link="body_link"/>
     <child link="imu_link"/>
-    <origin xyz="0.1 0 ${s1 + s5}" rpy="0 0 3.14159"/>
+    <origin xyz="0.1 0 ${s1 + s5}" rpy="0 0 0"/>
   </joint>
   <link name="imu_link">

Commit message: Refactor URDF structure to add base_link and adjust joint definitions for consistency with MOLA requirements

File: src/ros_gz_description/models/xacro_test/test.urdf.xacro (robot description, xacro)
@@ -58,6 +58,17 @@
   <!-- ==================== LINKS AND JOINTS ==================== -->
   <link name="base_footprint"/>
+  <!-- base_link sits at the same pose as base_footprint (z=0).
+       Required so MOLA (and other REP-105 tools) can resolve a
+       'base_link' frame.  Keeping the offset at zero means EKF
+       (which moves base_footprint) and MOLA (which expects to see
+       odom->base_link) stay numerically consistent. -->
+  <link name="base_link"/>
+  <joint name="base_link_joint" type="fixed">
+    <parent link="base_footprint"/>
+    <child link="base_link"/>
+    <origin xyz="0 0 0" rpy="0 0 0"/>
+  </joint>
   <joint name="body_link_joint" type="fixed">
-    <parent link="base_footprint"/>
+    <parent link="base_link"/>
     <child link="body_link"/>
   </joint>

Commit message: Update odometry frame references to use base_link for consistency with MOLA requirements

File: src/ros_gz_description/models/xacro_test/test.urdf.xacro (robot description, xacro)
@@ -57,16 +57,12 @@
   </xacro:macro>
   <!-- ==================== LINKS AND JOINTS ==================== -->
-  <link name="base_footprint"/>
-  <!-- base_link sits at the same pose as base_footprint (z=0).
-       Required so MOLA (and other REP-105 tools) can resolve a
-       'base_link' frame.  Keeping the offset at zero means EKF
-       (which moves base_footprint) and MOLA (which expects to see
-       odom->base_link) stay numerically consistent. -->
+  <!-- base_link is the URDF root and the EKF base_link_frame.
+       MOLA's launcher always broadcasts a static TF
+         base_link -> base_footprint   (REP-120 direction)
+       so we must NOT also publish base_footprint -> base_link from
+       the URDF (that would create a TF loop).  base_footprint is
+       therefore not declared in the URDF -- it appears at runtime
+       as a child of base_link via MOLA's static broadcaster. -->
   <link name="base_link"/>
-  <joint name="base_link_joint" type="fixed">
-    <parent link="base_footprint"/>
-    <child link="base_link"/>
-    <origin xyz="0 0 0" rpy="0 0 0"/>
-  </joint>
   <joint name="body_link_joint" type="fixed">
     <parent link="base_link"/>

Commit message: Update RViz configuration and launch files for improved TF management and visualization

File: src/ros_gz_description/models/xacro_test/test.urdf.xacro (robot description, xacro)
@@ -57,11 +57,19 @@
   </xacro:macro>
   <!-- ==================== LINKS AND JOINTS ==================== -->
-  <!-- base_link is the URDF root and the EKF base_link_frame.
-       MOLA's launcher always broadcasts a static TF
-         base_link to base_footprint  (REP-120 direction),
-       so we must NOT also publish base_footprint to base_link from
-       the URDF (that would create a TF loop).  base_footprint is
-       therefore not declared in the URDF; it appears at runtime
-       as a child of base_link via MOLA's static broadcaster. -->
+  <!-- ============================================================
+       TF OWNERSHIP
+       ============================================================
+       map           <- mola_lidar_odometry  (REP-105)
+       odom          <- ekf_filter_node      (world_frame=odom,
+                                              base_link_frame=base_link)
+       base_link     <- URDF root (this link)
+       base_footprint <- mola's static broadcaster, child of base_link
+                         (do NOT declare it here -- declaring it would
+                         duplicate that static TF and trigger
+                         TF_REPEATED_DATA spam)
+       body_link, wheels, imu_link, camera_link, laser
+                     <- this URDF (all rigidly attached to base_link
+                        via body_link)
+       ============================================================ -->
   <link name="base_link"/>
   <joint name="body_link_joint" type="fixed">
@@ -225,24 +233,29 @@
     </collision>
   </gazebo>
-  <!-- HINGE LINK (Vippepunktet) -->
-  <joint name="lidar_joint" type="revolute">
-    <parent link="body_link"/>
-    <child link="lidar_hinge_link"/>
-    <origin xyz="0 0 ${s1+s5}" rpy="0 0 0"/>
-    <axis xyz="0 1 0"/> <!-- Vipper opp og ned om Y-aksen -->
-    <limit lower="-0.785398" upper="0.785398" effort="10.0" velocity="5.0"/> <!-- +/- 45 grader -->
-    <dynamics damping="0.1" friction="0.1"/>
-  </joint>
-  <link name="lidar_hinge_link">
-    <inertial>
-      <mass value="0.05"/>
-      <inertia ixx="0.0001" ixy="0" ixz="0" iyy="0.0001" iyz="0" izz="0.0001"/>
-    </inertial>
-  </link>
-  <!-- SENSOR LINK (Forskyvningen på 32mm over vippepunktet) -->
-  <joint name="lidar_sensor_joint" type="fixed">
-    <parent link="lidar_hinge_link"/>
+  <!-- ============================================================
+       LIDAR MOUNT  (rigid in URDF on purpose)
+       ============================================================
+       The LD06 sits on a hobby-servo cradle that physically nods
+       +/- 30 deg, but the lidar3d ROS node already de-tilts every
+       point using the live servo-angle feedback and publishes the
+       resulting 3D cloud in the LEVEL `body_link` frame.
+       Therefore the URDF must NOT also tilt `laser` independently
+       in TF -- doing that creates two uncorrelated copies of the
+       tilt motion: the cloud stays flat in body_link while the
+       URDF visual nods around it, and any small MOLA pitch wobble
+       then shows up as the entire world tilting under a level
+       robot in RViz.
+       Keep this joint FIXED.  If you ever want to visualise the
+       servo angle on its own, do it in a debug-only TF (e.g. a
+       separate `lidar_tilt_visual_link` driven by joint_states)
+       that nothing in the SLAM pipeline subscribes to.
+       ------------------------------------------------------------
+       Offset: hinge sits ${s1+s5} above body_link origin, sensor
+       optical centre is +32 mm above the hinge.
+       ------------------------------------------------------------ -->
+  <joint name="lidar_joint" type="fixed">
+    <parent link="body_link"/>
     <child link="laser"/>
-    <origin xyz="0 0 0.032" rpy="0 0 0"/> <!-- 32 mm opp (Z-aksen) -->
+    <origin xyz="0 0 ${s1+s5+0.032}" rpy="0 0 0"/>
   </joint>
   <link name="laser">

Commit message: restored to last working state

File: src/ros_gz_description/models/xacro_test/test.urdf.xacro (robot description, xacro)
@@ -57,19 +57,4 @@
   </xacro:macro>
   <!-- ==================== LINKS AND JOINTS ==================== -->
-  <!-- ============================================================
-       TF OWNERSHIP
-       ============================================================
-       map            <- mola_lidar_odometry  (REP-105)
-       odom           <- ekf_filter_node      (world_frame=odom,
-                                               base_link_frame=base_link)
-       base_link      <- URDF root (this link)
-       base_footprint <- mola's static broadcaster, child of base_link
-                         (do NOT declare it here; declaring it would
-                         duplicate that static TF and trigger
-                         TF_REPEATED_DATA spam)
-       body_link, wheels, imu_link, camera_link, laser
-                      <- this URDF (all rigidly attached to base_link
-                         via body_link)
-       ============================================================ -->
   <link name="base_footprint"/>
   <joint name="body_link_joint" type="fixed">
@@ -233,29 +218,24 @@
     </collision>
   </gazebo>
-  <!-- ============================================================
-       LIDAR MOUNT  (rigid in URDF on purpose)
-       ============================================================
-       The LD06 sits on a hobby-servo cradle that physically nods
-       +/- 30 deg, but the lidar3d ROS node already de-tilts every
-       point using the live servo-angle feedback and publishes the
-       resulting 3D cloud in the LEVEL `body_link` frame.
-       Therefore the URDF must NOT also tilt `laser` independently
-       in TF; doing that creates two uncorrelated copies of the
-       tilt motion: the cloud stays flat in body_link while the
-       URDF visual nods around it, and any small MOLA pitch wobble
-       then shows up as the entire world tilting under a level
-       robot in RViz.
-       Keep this joint FIXED.  If you ever want to visualise the
-       servo angle on its own, do it in a debug-only TF (e.g. a
-       separate `lidar_tilt_visual_link` driven by joint_states)
-       that nothing in the SLAM pipeline subscribes to.
-       ============================================================
-       Offset: hinge sits ${s1+s5} above body_link origin, sensor
-       optical centre is +32 mm above the hinge.
-       ============================================================ -->
-  <joint name="lidar_joint" type="fixed">
-    <parent link="body_link"/>
+  <!-- HINGE LINK (Vippepunktet) -->
+  <joint name="lidar_joint" type="revolute">
+    <parent link="body_link"/>
+    <child link="lidar_hinge_link"/>
+    <origin xyz="0 0 ${s1+s5}" rpy="0 0 0"/>
+    <axis xyz="0 1 0"/> <!-- Vipper opp og ned om Y-aksen -->
+    <limit lower="-0.785398" upper="0.785398" effort="10.0" velocity="5.0"/> <!-- +/- 45 grader -->
+    <dynamics damping="0.1" friction="0.1"/>
+  </joint>
+  <link name="lidar_hinge_link">
+    <inertial>
+      <mass value="0.05"/>
+      <inertia ixx="0.0001" ixy="0" ixz="0" iyy="0.0001" iyz="0" izz="0.0001"/>
+    </inertial>
+  </link>
+  <!-- SENSOR LINK (Forskyvningen på 32mm over vippepunktet) -->
+  <joint name="lidar_sensor_joint" type="fixed">
+    <parent link="lidar_hinge_link"/>
     <child link="laser"/>
-    <origin xyz="0 0 ${s1+s5+0.032}" rpy="0 0 0"/>
+    <origin xyz="0 0 0.032" rpy="0 0 0"/> <!-- 32 mm opp (Z-aksen) -->
   </joint>
   <link name="laser">
