Commit message: Update joint orientation for base_footprint to base_link connection in URDF

File: src/GregorURDF/urdf/gregor.urdf (robot description, URDF)
Before this commit: robot gregor, 21 links, 20 joints
Joints:
- joint base_footprint_to_base_link: origin xyz=0 0 0.025 rpy=0 0 0 -> xyz=0 0 0.025 rpy=0 0 -1.5708

Commit message: Fix joint orientation for base_footprint to base_link connection in URDF

File: src/GregorURDF/urdf/gregor.urdf (robot description, URDF)
Before this commit: robot gregor, 21 links, 20 joints
Joints:
- joint base_footprint_to_base_link: origin xyz=0 0 0.025 rpy=0 0 -1.5708 -> xyz=0 0 0.025 rpy=0 0 0

Commit message: Add URDF model for the 'gregor' robot
- Created a comprehensive URDF file defining the robot structure, including links and joints.
- Defined inertial properties, visual representations, and collision geometries for various components such as the upper level, battery, camera, and range sensors.
- Established fixed and continuous joints to connect the robot's components, ensuring accurate representation of the robot's kinematics.
- Included detailed specifications for each link, including mass, inertia, and mesh file paths for visual representation.

File: src/GregorURDF/urdf/gregor.urdf (robot description, URDF)
Before this commit: robot gregor, 21 links, 20 joints
Joints:
- removed joint base_link_to_battery
- removed joint base_link_to_motor_fl
- removed joint base_link_to_motor_fr
- removed joint base_link_to_motor_rl
- removed joint base_link_to_motor_rr
- removed joint base_link_to_range_front
- removed joint base_link_to_range_rear
- removed joint base_link_to_upper_level
- removed joint lidar_mount_to_laser
- removed joint motor_fl_to_wheel_fl
- removed joint motor_fr_to_wheel_fr
- removed joint motor_rl_to_wheel_rl
- removed joint motor_rr_to_wheel_rr
- removed joint upper_level_to_camera
- removed joint upper_level_to_imu
- removed joint upper_level_to_lidar_mount
- removed joint upper_level_to_range_left
- removed joint upper_level_to_range_right
- removed joint upper_level_to_thermal_camera
- added joint Chassie_Rigid-1: type fixed, parent base_link, child battery_link, origin xyz=0.00015423000372526423 -0.007561000130385147 -1.4210854715202004e-16 rpy=3.141592653589793 6.1584619237316516e-33 -1.5707963267948966
- added joint Chassie_Rigid-11: type fixed, parent base_link, child range_rear_link, origin xyz=-0.012835639996274736 0.12549999986961483 -0.00800000000000015 rpy=3.141592653589793 6.1584619237316516e-33 -1.5707963267948966
- added joint Chassie_Rigid-2: type fixed, parent base_link, child upper_level_link, origin xyz=0.00015423000372526423 -0.007561000130385147 0.007999999999999856 rpy=-3.2526065174564526e-19 6.1584619237316516e-33 -1.5707963267948966
- added joint Chassie_Rigid-21: type fixed, parent base_link, child motor_rr_link, origin xyz=-0.04999999999627474 0.06499999986961483 -0.019000000000000152 rpy=1.5707963267948966 -1.5707963267948966 0
- added joint Chassie_Rigid-23: type fixed, parent base_link, child motor_fr_link, origin xyz=-0.04999999999627474 -0.08000000013038511 -0.019000000000000152 rpy=-1.5707963267948968 -1.5707963267948966 0
- added joint Chassie_Rigid-24: type fixed, parent base_link, child motor_fl_link, origin xyz=0.05033753000372526 -0.08010768013038512 -0.019000000000000152 rpy=1.5707963267948966 -1.5707963267948966 0
- added joint Chassie_Rigid-25: type fixed, parent base_link, child motor_rl_link, origin xyz=0.050354650003725264 0.06471500986961483 -0.019000000000000152 rpy=1.5707963267948966 -1.5707963267948966 0
- added joint Chassie_Rigid-9: type fixed, parent base_link, child range_front_link, origin xyz=0.013000710003725262 -0.14062201013038508 -0.005000000000000142 rpy=-3.2526065174564526e-19 6.1584619237316516e-33 -1.5707963267948966
- added joint LiDAR-Mount_Rigid-4: type fixed, parent lidar_mount_link, child laser, origin xyz=0.006150000000000003 3.469446951953614e-20 -2.1069999999999702e-05 rpy=1.102916357619544e-47 1.570796326794895 0
- added joint Motor-FL_Revolute-28: type continuous, parent motor_fl_link, child wheel_fl_link, origin xyz=0.0 0.0 0.0 rpy=-2.660190735689466e-33 -0.0 0.0, axis 0.0 1.0 2.4034014453635364e-47
- added joint Motor-FR_Revolute-27: type continuous, parent motor_fr_link, child wheel_fr_link, origin xyz=0.0 0.0 0.0 rpy=3.141592653589793 -0.0 0.0, axis 0.0 -1.0 2.1209945128196103e-51
- added joint Motor-RL_Revolute-26: type continuous, parent motor_rl_link, child wheel_rl_link, origin xyz=0.0 0.0 0.0 rpy=3.141592653589793 7.022514532037904e-97 3.503246160812043e-46, axis -3.503246160812043e-46 1.0 2.495984093634733e-46
- added joint Motor-RR_Revolute-22: type continuous, parent motor_rr_link, child wheel_rr_link, origin xyz=0.0 0.0 0.0 rpy=3.141592653589793 -0.0 0.0, axis 0.0 -1.0 -4.022647846648095e-51
- added joint Upper-Level_Revolute-3: type continuous, parent upper_level_link, child lidar_mount_link, origin xyz=4.479000000000011e-05 -3.5119999999999996e-05 0.08375145 rpy=-1.6930901125533616e-15 -1.5707963267948966 0, axis 9.398538128609942e-32 -0.9999999999999996 -1.6930901125533608e-15
- added joint Upper-Level_Rigid-29: type fixed, parent upper_level_link, child range_right_link, origin xyz=0.01349606 -0.08622216999999999 -0.018 rpy=0.0 -0.0 0.0
- added joint Upper-Level_Rigid-5: type fixed, parent upper_level_link, child camera_link, origin xyz=0.057249999999999995 -0.03049246 0.056499999999999995 rpy=1.570796326794901 -0.0 0.0
- added joint Upper-Level_Rigid-6: type fixed, parent upper_level_link, child thermal_camera_link, origin xyz=0.057249999999999995 0.02750754 0.056499999999999995 rpy=1.5707963267948966 -0.0 0.0
- added joint Upper-Level_Rigid-7: type fixed, parent upper_level_link, child imu_link, origin xyz=0.0 0.0 0.04035000000000001 rpy=0.0 -0.0 0.0
- added joint Upper-Level_Rigid-8: type fixed, parent upper_level_link, child range_left_link, origin xyz=-0.012 0.085 -0.014802099999999997 rpy=0.0 -0.0 0.0

Commit message: Fix joint orientation for Upper-Level_Rigid-7 in URDF

File: src/GregorURDF/urdf/gregor.urdf (robot description, URDF)
Before this commit: robot gregor, 21 links, 20 joints
Joints:
- joint Upper-Level_Rigid-7: origin xyz=0.0 0.0 0.04035000000000001 rpy=0.0 -0.0 0.0 -> xyz=0.0 0.0 0.04035000000000001 rpy=0.0 -0.0 -1.5708

Commit message: Fix joint orientation for Upper-Level_Rigid-7 and base_footprint to base_link in URDF

File: src/GregorURDF/urdf/gregor.urdf (robot description, URDF)
Before this commit: robot gregor, 21 links, 20 joints
Joints:
- joint Upper-Level_Rigid-7: origin xyz=0.0 0.0 0.04035000000000001 rpy=0.0 -0.0 -1.5708 -> xyz=0.0 0.0 0.04035000000000001 rpy=0.0 -0.0 0.0
- joint base_footprint_to_base_link: origin xyz=0 0 0.025 rpy=0 0 0 -> xyz=0 0 0.025 rpy=0 0 1.5707963267948966

Commit message: Change joint type of Upper-Level_Revolute-3 from continuous to fixed

File: src/GregorURDF/urdf/gregor.urdf (robot description, URDF)
Before this commit: robot gregor, 21 links, 20 joints
Joints:
- joint Upper-Level_Revolute-3: type continuous -> fixed

Commit message: Add 3D mapping configuration and launch files for simulation and real robot

File: src/GregorURDF/urdf/gregor.urdf (robot description, URDF)
Before this commit: robot gregor, 21 links, 20 joints
Links:
- link range_right_link: geometry collision mesh filename=package://gregor_description/meshes/Avstands-sensor-høyre.s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 scale=0.001 0.001 0.001; visual mesh filename=package://gregor_description/meshes/Avstands-sensor-hoyre.s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 scale=0.001 0.001 0.001
Joints:
- joint Motor-FL_Revolute-28: limit (none) -> effort=50000 velocity=10
- joint Motor-FR_Revolute-27: limit (none) -> effort=50000 velocity=10
- joint Motor-RL_Revolute-26: limit (none) -> effort=50000 velocity=10
- joint Motor-RR_Revolute-22: limit (none) -> effort=50000 velocity=10
- joint Upper-Level_Revolute-3: limit (none) -> lower=-0.785398 upper=0.785398 effort=10.0 velocity=5.0; type continuous -> revolute
- joint base_footprint_to_base_link: origin xyz=0 0 0.025 rpy=0 0 1.5707963267948966 -> xyz=0 0 0.025 rpy=0 0 0

Commit message: Refactor lidar3D node for improved simulation handling and update launch configurations

File: src/GregorURDF/urdf/gregor.urdf (robot description, URDF)
Before this commit: robot gregor, 21 links, 20 joints
Links:
- link range_right_link: geometry collision mesh filename=package://gregor_description/meshes/Avstands-sensor-hoyre.s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 scale=0.001 0.001 0.001; visual mesh filename=package://gregor_description/meshes/Avstands-sensor-hoyre.s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 scale=0.001 0.001 0.001
Joints:
- joint LiDAR-Mount_Rigid-4: origin xyz=0.006150000000000003 3.469446951953614e-20 -2.1069999999999702e-05 rpy=1.102916357619544e-47 1.570796326794895 0 -> xyz=0 0 0.00615 rpy=0 0 3.141592653589793
- joint Upper-Level_Revolute-3: axis 9.398538128609942e-32 -0.9999999999999996 -1.6930901125533608e-15 -> 1 0 0; origin xyz=4.479000000000011e-05 -3.5119999999999996e-05 0.08375145 rpy=-1.6930901125533616e-15 -1.5707963267948966 0 -> xyz=0 0 0.08375145 rpy=0 0 1.5707963267948966

File: src/ros_gz_example_gazebo/worlds/test_xacro.sdf.xacro (robot description, xacro)
@@ -140,9 +140,4 @@
     </include>
     -->
-    <include>
-      <uri>model://xacro_test</uri>
-      <name>test_robot</name>
-      <pose>0 0 0.15 0 0 0</pose>
-    </include>
   </world>
 </sdf>

Commit message: Update URDF joint orientations and collision geometries for Mecanum wheels; enhance 3D mapping bridge configuration

File: src/GregorURDF/urdf/gregor.urdf (robot description, URDF)
Before this commit: robot gregor, 21 links, 20 joints
Links:
- link wheel_fl_link: geometry collision cylinder length=0.030 radius=0.0375; visual mesh filename=package://gregor_description/meshes/Mecanum-wheel-FL.stl scale=0.001 0.001 0.001
- link wheel_fr_link: geometry collision cylinder length=0.030 radius=0.0375; visual mesh filename=package://gregor_description/meshes/Mecanum-wheel-FR.stl scale=0.001 0.001 0.001
- link wheel_rl_link: geometry collision cylinder length=0.030 radius=0.0375; visual mesh filename=package://gregor_description/meshes/Mecanum-wheel-RL.stl scale=0.001 0.001 0.001
- link wheel_rr_link: geometry collision cylinder length=0.030 radius=0.0375; visual mesh filename=package://gregor_description/meshes/Mecanum-wheel-RR.stl scale=0.001 0.001 0.001
Joints:
- joint Motor-FL_Revolute-28: axis 0.0 1.0 2.4034014453635364e-47 -> 0.0 -1.0 0.0; origin xyz=0.0 0.0 0.0 rpy=-2.660190735689466e-33 -0.0 0.0 -> xyz=0.0 0.0 0.0 rpy=0.0 0.0 0.0
- joint Motor-FR_Revolute-27: axis 0.0 -1.0 2.1209945128196103e-51 -> 0.0 -1.0 0.0; origin xyz=0.0 0.0 0.0 rpy=3.141592653589793 -0.0 0.0 -> xyz=0.0 0.0 0.0 rpy=3.141592653589793 0.0 0.0
- joint Motor-RL_Revolute-26: axis -3.503246160812043e-46 1.0 2.495984093634733e-46 -> 0.0 1.0 0.0; origin xyz=0.0 0.0 0.0 rpy=3.141592653589793 7.022514532037904e-97 3.503246160812043e-46 -> xyz=0.0 0.0 0.0 rpy=3.141592653589793 0.0 0.0
- joint Motor-RR_Revolute-22: axis 0.0 -1.0 -4.022647846648095e-51 -> 0.0 1.0 0.0; origin xyz=0.0 0.0 0.0 rpy=3.141592653589793 -0.0 0.0 -> xyz=0.0 0.0 0.0 rpy=3.141592653589793 0.0 0.0
- joint base_footprint_to_base_link: origin xyz=0 0 0.025 rpy=0 0 0 -> xyz=0 0 0.025 rpy=0 0 1.5707963

Commit message: fixed mecanum drive in sim!

File: src/GregorURDF/urdf/gregor.urdf (robot description, URDF)
Before this commit: robot gregor, 21 links, 20 joints
Links:
- link base_link: geometry visual mesh filename=package://gregor_description/meshes/Chassie.stl scale=0.001 0.001 0.001
- link battery_link: geometry visual mesh filename=package://gregor_description/meshes/Battery.stl scale=0.001 0.001 0.001
- link camera_link: geometry visual mesh filename=package://gregor_description/meshes/RGB-Camera.stl scale=0.001 0.001 0.001
- link imu_link: geometry visual mesh filename=package://gregor_description/meshes/IMU.stl scale=0.001 0.001 0.001
- link laser: geometry visual mesh filename=package://gregor_description/meshes/LD06_LiDAR.stl scale=0.001 0.001 0.001
- link lidar_mount_link: geometry visual mesh filename=package://gregor_description/meshes/LiDAR-Mount.stl scale=0.001 0.001 0.001
- link motor_fl_link: geometry visual mesh filename=package://gregor_description/meshes/Motor-FL.stl scale=0.001 0.001 0.001
- link motor_fr_link: geometry visual mesh filename=package://gregor_description/meshes/Motor-FR.stl scale=0.001 0.001 0.001
- link motor_rl_link: geometry visual mesh filename=package://gregor_description/meshes/Motor-RL.stl scale=0.001 0.001 0.001
- link motor_rr_link: geometry visual mesh filename=package://gregor_description/meshes/Motor-RR.stl scale=0.001 0.001 0.001
- link range_front_link: geometry visual mesh filename=package://gregor_description/meshes/Avstands-sensor-fremme.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 scale=0.001 0.001 0.001
- link range_left_link: geometry visual mesh filename=package://gregor_description/meshes/Avstands-sensor-venstre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 scale=0.001 0.001 0.001
- link range_rear_link: geometry visual mesh filename=package://gregor_description/meshes/Avstands-sensor-bak.stl scale=0.001 0.001 0.001
- link range_right_link: geometry visual mesh filename=package://gregor_description/meshes/Avstands-sensor-hoyre.s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 scale=0.001 0.001 0.001
- link thermal_camera_link: geometry visual mesh filename=package://gregor_description/meshes/Thermal-camera.stl scale=0.001 0.001 0.001
- link upper_level_link: geometry visual mesh filename=package://gregor_description/meshes/Upper-Level.stl scale=0.001 0.001 0.001
- link wheel_fl_link: geometry collision sphere radius=0.0375; visual mesh filename=package://gregor_description/meshes/Mecanum-wheel-FL.stl scale=0.001 0.001 0.001
- link wheel_fr_link: geometry collision sphere radius=0.0375; visual mesh filename=package://gregor_description/meshes/Mecanum-wheel-FR.stl scale=0.001 0.001 0.001
- link wheel_rl_link: geometry collision sphere radius=0.0375; visual mesh filename=package://gregor_description/meshes/Mecanum-wheel-RL.stl scale=0.001 0.001 0.001
- link wheel_rr_link: geometry collision sphere radius=0.0375; visual mesh filename=package://gregor_description/meshes/Mecanum-wheel-RR.stl scale=0.001 0.001 0.001
Joints:
- joint base_footprint_to_base_link: origin xyz=0 0 0.025 rpy=0 0 1.5707963 -> xyz=0 0 0.025 rpy=0 0 1.5707963267948966

File: src/ros_gz_example_gazebo/worlds/test_xacro.sdf.xacro (robot description, xacro)
@@ -98,4 +98,12 @@
         <collision name="collision">
           <geometry><plane><normal>0 0 1</normal></plane></geometry>
+          <surface>
+            <friction>
+              <ode>
+                <mu>50</mu>
+                <mu2>50</mu2>
+              </ode>
+            </friction>
+          </surface>
         </collision>
         <visual name="visual">
