Commit message: Update mapping parameters and launch configurations for Gregor robot
- Changed base frame from 'base_link' to 'base_footprint' in mapper_params_online_async.yaml for improved mapping accuracy.
- Updated frame IDs in gregor_real.launch.py:
  - Changed LiDAR frame ID from 'LD06_LiDAR' to 'laser_link'.
  - Changed camera frame ID from 'RGB-Camera' to 'camera_link'.
- Added a backup of the URDF file for the Gregor robot, ensuring version control and easier rollback if needed.

Co-authored-by: Copilot <copilot@github.com>

File: src/GregorURDF/urdf/gregor.urdf (robot description, URDF)
Before this commit: robot Gergor, 20 links, 19 joints
Links:
- removed link Avstands-sensor-bak
- removed link Avstands-sensor-fremme
- removed link Avstands-sensor-høyre
- removed link Avstands-sensor-venstre
- removed link Battery
- removed link Chassie
- removed link IMU
- removed link LD06_LiDAR
- removed link LiDAR-Mount
- removed link Mecanum-wheel-FL
- removed link Mecanum-wheel-FR
- removed link Mecanum-wheel-RL
- removed link Mecanum-wheel-RR
- removed link Motor-FL
- removed link Motor-FR
- removed link Motor-RL
- removed link Motor-RR
- removed link RGB-Camera
- removed link Thermal-camera
- removed link Upper-Level
- added link base_footprint
- added link base_link, mass 0.29216485565837275; collision mesh filename=package://gregor_description/meshes/Chassie.stl scale=0.001 0.001 0.001; visual mesh filename=package://gregor_description/meshes/Chassie.stl scale=0.001 0.001 0.001
- added link battery_link, mass 0.09697089693767996; collision mesh filename=package://gregor_description/meshes/Battery.stl scale=0.001 0.001 0.001; visual mesh filename=package://gregor_description/meshes/Battery.stl scale=0.001 0.001 0.001
- added link camera_link, mass 0.00705801985514185; collision mesh filename=package://gregor_description/meshes/RGB-Camera.stl scale=0.001 0.001 0.001; visual mesh filename=package://gregor_description/meshes/RGB-Camera.stl scale=0.001 0.001 0.001
- added link imu_link, mass 0.0003552000152170653; collision mesh filename=package://gregor_description/meshes/IMU.stl scale=0.001 0.001 0.001; visual mesh filename=package://gregor_description/meshes/IMU.stl scale=0.001 0.001 0.001
- added link laser_link, mass 0.07569091272999597; collision mesh filename=package://gregor_description/meshes/LD06_LiDAR.stl scale=0.001 0.001 0.001; visual mesh filename=package://gregor_description/meshes/LD06_LiDAR.stl scale=0.001 0.001 0.001
- added link lidar_mount_link, mass 0.025423989422360332; collision mesh filename=package://gregor_description/meshes/LiDAR-Mount.stl scale=0.001 0.001 0.001; visual mesh filename=package://gregor_description/meshes/LiDAR-Mount.stl scale=0.001 0.001 0.001
- added link motor_fl_link, mass 0.15441088816550527; collision mesh filename=package://gregor_description/meshes/Motor-FL.stl scale=0.001 0.001 0.001; visual mesh filename=package://gregor_description/meshes/Motor-FL.stl scale=0.001 0.001 0.001
- added link motor_fr_link, mass 0.15441088816550527; collision mesh filename=package://gregor_description/meshes/Motor-FR.stl scale=0.001 0.001 0.001; visual mesh filename=package://gregor_description/meshes/Motor-FR.stl scale=0.001 0.001 0.001
- added link motor_rl_link, mass 0.15441088816550527; collision mesh filename=package://gregor_description/meshes/Motor-RL.stl scale=0.001 0.001 0.001; visual mesh filename=package://gregor_description/meshes/Motor-RL.stl scale=0.001 0.001 0.001
- added link motor_rr_link, mass 0.15441088816550527; collision mesh filename=package://gregor_description/meshes/Motor-RR.stl scale=0.001 0.001 0.001; visual mesh filename=package://gregor_description/meshes/Motor-RR.stl scale=0.001 0.001 0.001
- added link range_front_link, mass 0.011156887500000002; collision mesh filename=package://gregor_description/meshes/Avstands-sensor-fremme.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 scale=0.001 0.001 0.001; visual mesh filename=package://gregor_description/meshes/Avstands-sensor-fremme.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 scale=0.001 0.001 0.001
- added link range_left_link, mass 0.0111568875; collision mesh filename=package://gregor_description/meshes/Avstands-sensor-venstre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 scale=0.001 0.001 0.001; visual mesh filename=package://gregor_description/meshes/Avstands-sensor-venstre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 scale=0.001 0.001 0.001
- added link range_rear_link, mass 0.011156887500000002; collision mesh filename=package://gregor_description/meshes/Avstands-sensor-bak.stl scale=0.001 0.001 0.001; visual mesh filename=package://gregor_description/meshes/Avstands-sensor-bak.stl scale=0.001 0.001 0.001
- added link range_right_link, mass 0.0111568875; collision mesh filename=package://gregor_description/meshes/Avstands-sensor-høyre.s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 scale=0.001 0.001 0.001; visual mesh filename=package://gregor_description/meshes/Avstands-sensor-høyre.s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 scale=0.001 0.001 0.001
- added link thermal_camera_link, mass 0.0030870822826619742; collision mesh filename=package://gregor_description/meshes/Thermal-camera.stl scale=0.001 0.001 0.001; visual mesh filename=package://gregor_description/meshes/Thermal-camera.stl scale=0.001 0.001 0.001
- added link upper_level_link, mass 0.13651212208139799; collision mesh filename=package://gregor_description/meshes/Upper-Level.stl scale=0.001 0.001 0.001; visual mesh filename=package://gregor_description/meshes/Upper-Level.stl scale=0.001 0.001 0.001
- added link wheel_fl_link, mass 0.1511892944710378; collision mesh filename=package://gregor_description/meshes/Mecanum-wheel-FL.stl scale=0.001 0.001 0.001; visual mesh filename=package://gregor_description/meshes/Mecanum-wheel-FL.stl scale=0.001 0.001 0.001
- added link wheel_fr_link, mass 0.1511892944710378; collision mesh filename=package://gregor_description/meshes/Mecanum-wheel-FR.stl scale=0.001 0.001 0.001; visual mesh filename=package://gregor_description/meshes/Mecanum-wheel-FR.stl scale=0.001 0.001 0.001
- added link wheel_rl_link, mass 0.1511892944710378; collision mesh filename=package://gregor_description/meshes/Mecanum-wheel-RL.stl scale=0.001 0.001 0.001; visual mesh filename=package://gregor_description/meshes/Mecanum-wheel-RL.stl scale=0.001 0.001 0.001
- added link wheel_rr_link, mass 0.1511892944710378; collision mesh filename=package://gregor_description/meshes/Mecanum-wheel-RR.stl scale=0.001 0.001 0.001; visual mesh filename=package://gregor_description/meshes/Mecanum-wheel-RR.stl scale=0.001 0.001 0.001
Joints:
- removed joint Chassie_Rigid-1
- removed joint Chassie_Rigid-11
- removed joint Chassie_Rigid-2
- removed joint Chassie_Rigid-21
- removed joint Chassie_Rigid-23
- removed joint Chassie_Rigid-24
- removed joint Chassie_Rigid-25
- removed joint Chassie_Rigid-9
- removed joint LiDAR-Mount_Rigid-4
- removed joint Motor-FL_Revolute-28
- removed joint Motor-FR_Revolute-27
- removed joint Motor-RL_Revolute-26
- removed joint Motor-RR_Revolute-22
- removed joint Upper-Level_Revolute-3
- removed joint Upper-Level_Rigid-29
- removed joint Upper-Level_Rigid-5
- removed joint Upper-Level_Rigid-6
- removed joint Upper-Level_Rigid-7
- removed joint Upper-Level_Rigid-8
- added joint base_footprint_to_base_link: type fixed, parent base_footprint, child base_link, origin xyz=0 0 0.025 rpy=0 0 0
- added joint base_link_to_battery: type fixed, parent base_link, child battery_link, origin xyz=0.00015423000372529028 -0.007561000130385162 -1.509903313490213e-16 rpy=3.141592653589793 3.252606517456514e-19 -7.888609052210118e-31
- added joint base_link_to_motor_fl: type fixed, parent base_link, child motor_fl_link, origin xyz=0.05033753000372532 -0.08010768013038516 -0.01900000000000016 rpy=3.141592653589793 -1.5707963267948966 0
- added joint base_link_to_motor_fr: type fixed, parent base_link, child motor_fr_link, origin xyz=-0.04999999999627474 -0.08000000013038516 -0.01900000000000016 rpy=-7.888609052210122e-31 -1.5707963267948966 0
- added joint base_link_to_motor_rl: type fixed, parent base_link, child motor_rl_link, origin xyz=0.05035465000372532 0.06471500986961484 -0.01900000000000016 rpy=3.141592653589793 -1.5707963267948966 0
- added joint base_link_to_motor_rr: type fixed, parent base_link, child motor_rr_link, origin xyz=-0.04999999999627474 0.06499999986961484 -0.01900000000000016 rpy=3.141592653589793 -1.5707963267948966 0
- added joint base_link_to_range_front: type fixed, parent base_link, child range_front_link, origin xyz=0.013000710003725298 -0.14062201013038517 -0.005000000000000151 rpy=-2.563333722837743e-49 3.252606517456514e-19 -7.888609052210118e-31
- added joint base_link_to_range_rear: type fixed, parent base_link, child range_rear_link, origin xyz=-0.012835639996274717 0.12549999986961485 -0.008000000000000158 rpy=3.141592653589793 3.252606517456514e-19 -7.888609052210118e-31
- added joint base_link_to_upper_level: type fixed, parent base_link, child upper_level_link, origin xyz=0.00015423000372529028 -0.007561000130385162 0.007999999999999848 rpy=-2.563333722837743e-49 3.252606517456514e-19 -7.888609052210118e-31
- added joint lidar_mount_to_laser: type fixed, parent lidar_mount_link, child laser_link, origin xyz=0.0061499999999999845 -2.106999999999998e-05 3.1225022567582527e-19 rpy=-1.0868129502412381e-47 1.570796326794895 0
- added joint motor_fl_to_wheel_fl: type continuous, parent motor_fl_link, child wheel_fl_link, origin xyz=0.0 0.0 0.0 rpy=-7.915210959567012e-31 -3.0814879110195774e-33 3.4211388289180104e-49, axis -3.0814879110195774e-33 7.915210959567012e-31 -1.0
- added joint motor_fr_to_wheel_fr: type continuous, parent motor_fr_link, child wheel_fr_link, origin xyz=0.0 0.0 0.0 rpy=3.141592653589793 -0.0 -3.4211388289180104e-49, axis 0.0 -2.9999493436745292e-33 1.0
- added joint motor_rl_to_wheel_rl: type continuous, parent motor_rl_link, child wheel_rl_link, origin xyz=0.0 0.0 0.0 rpy=3.141592653589793 -4.930380657631324e-32 3.4211388289180104e-49, axis 4.930380657631324e-32 3.857676143488164e-45 -1.0
- added joint motor_rr_to_wheel_rr: type continuous, parent motor_rr_link, child wheel_rr_link, origin xyz=0.0 0.0 0.0 rpy=3.141592653589793 -0.0 1.7105694144590052e-48, axis -0.0 -3.942138089887358e-34 1.0
- added joint upper_level_to_camera: type fixed, parent upper_level_link, child camera_link, origin xyz=-0.03049246 -0.057249999999999995 0.056499999999999995 rpy=1.570796326794901 -0.0 1.6472184286297693e-83
- added joint upper_level_to_imu: type fixed, parent upper_level_link, child imu_link, origin xyz=0.0 0.0 0.04035000000000001 rpy=0.0 -0.0 1.6472184286297693e-83
- added joint upper_level_to_lidar_mount: type continuous, parent upper_level_link, child lidar_mount_link, origin xyz=-3.5119999999999996e-05 -4.479000000000011e-05 0.08375145 rpy=-1.6514567491299184e-15 -1.5707963267948966 0, axis -5.551115123125929e-17 -1.6514567491299192e-15 1.0000000000000004
- added joint upper_level_to_range_left: type fixed, parent upper_level_link, child range_left_link, origin xyz=0.085 0.012 -0.014802099999999997 rpy=0.0 -0.0 1.6472184286297693e-83
- added joint upper_level_to_range_right: type fixed, parent upper_level_link, child range_right_link, origin xyz=-0.08622216999999999 -0.01349606 -0.018 rpy=0.0 -0.0 1.6472184286297693e-83
- added joint upper_level_to_thermal_camera: type fixed, parent upper_level_link, child thermal_camera_link, origin xyz=0.02750754 -0.057249999999999995 0.056499999999999995 rpy=1.5707963267948966 -0.0 1.6472184286297693e-83

Commit message: Rename 'laser_link' to 'laser' in URDF and update launch configuration accordingly
Co-authored-by: Copilot <copilot@github.com>

File: src/GregorURDF/urdf/gregor.urdf (robot description, URDF)
Before this commit: robot gregor, 21 links, 20 joints
Links:
- removed link laser_link
- added link laser, mass 0.07569091272999597; collision mesh filename=package://gregor_description/meshes/LD06_LiDAR.stl scale=0.001 0.001 0.001; visual mesh filename=package://gregor_description/meshes/LD06_LiDAR.stl scale=0.001 0.001 0.001
Joints:
- joint lidar_mount_to_laser: child laser_link -> laser

Commit message: revert(gregor.urdf): keep Mola's revolute tilt joint, not main's fixed
The merge took main's type="fixed" + CAD-exported origin for
Upper-Level_Revolute-3. The Mola branch already had a more
deliberate version: type="revolute" with the documented
"yaw=+π/2 cancels upper_level_link's -π/2 yaw" geometry. That's
the working version we want to keep.

Co-Authored-By: Claude Opus 4.7 <noreply@anthropic.com>

File: src/GregorURDF/urdf/gregor.urdf (robot description, URDF)
Before this commit: robot gregor, 21 links, 20 joints
Joints:
- joint Upper-Level_Revolute-3: origin xyz=4.479000000000011e-05 -3.5119999999999996e-05 0.08375145 rpy=-1.6930901125533616e-15 -1.5707963267948966 0 -> xyz=0 0 0.08375145 rpy=0 0 1.5707963267948966; type fixed -> revolute
