Commit message: Enhance 3D mapping and EKF configurations for improved performance
- Adjusted lidar3d parameters in 3d_mapping.yaml to narrow tilt sweep to ±20° and increased sweep period to 0.5s for better body motion handling during turns.
- Updated EKF settings in ekf_imu.yaml to increase frequency from 10Hz to 50Hz, aligning with sensor output rates for smoother motion prior interpolation.
- Modified 3d_mapping_bridge.yaml to clarify the handling of odom→base_footprint TF, ensuring no conflicts with the EKF.
- Enhanced ekf.yaml to improve odometry and IMU integration, increasing frequency to 50Hz and refining configuration for better state estimation.
- Updated 3D mapping launch file (3dMapping.launch.py) to include EKF node and optional MOLA-LO integration for live SLAM, with a bag recorder for offline processing.
- Introduced mola_lo.launch.py for live MOLA-LO operation, ensuring consistent state estimation across simulation and real robot scenarios.
- Updated package.xml to include dependencies for MOLA state estimation packages.
- Adjusted test_xacro.sdf.xacro to modify arena size and ensure proper IMU sensor publishing for EKF functionality.

File: src/ros_gz_example_gazebo/worlds/test_xacro.sdf.xacro (robot description, xacro)
@@ -2,5 +2,5 @@
 <sdf version="1.8" xmlns:xacro="http://www.ros.org/wiki/xacro">
   <!-- Parametere -->
-  <xacro:property name="arena_size" value="10.0"/>
+  <xacro:property name="arena_size" value="5.0"/>
   <xacro:property name="wall_t" value="0.2"/>
   <xacro:property name="wall_h" value="1.0"/>
@@ -80,4 +80,8 @@
     <plugin filename="gz-sim-scene-broadcaster-system" name="gz::sim::systems::SceneBroadcaster"/>
     <plugin filename="gz-sim-sensors-system" name="gz::sim::systems::Sensors"/>
+    <!-- Required for the URDF's <sensor type="imu"> on imu_link to publish.
+         Without this the sensor element is parsed but no /imu messages are
+         emitted, which silently breaks the EKF in 3dMapping.launch.py. -->
+    <plugin filename="gz-sim-imu-system" name="gz::sim::systems::Imu"/>
     <light type="directional" name="sun">
       <cast_shadows>true</cast_shadows>
@@ -123,10 +127,10 @@
     <xacro:wall name="wall_west"  x="${-arena_size/2.0}" y="0" yaw="0" sx="${wall_t}" sy="${arena_size}" sz="${wall_h}"/>
     <!-- Interne vegger / rom -->
-    <!-- Vertikal vegg ved x = -1.5, med døråpning rundt y = 0 -->
-    <xacro:wall name="room_v_left_top" x="-1.5" y="2.0"  yaw="0" sx="${wall_t}" sy="3.0" sz="${wall_h}"/>
-    <xacro:wall name="room_v_left_bot" x="-1.5" y="-2.0" yaw="0" sx="${wall_t}" sy="3.0" sz="${wall_h}"/>
-    <!-- Vertikal vegg ved x = 1.8, med døråpning rundt y = -1 -->
-    <xacro:wall name="room_v_right_top" x="1.8" y="2.3"  yaw="0" sx="${wall_t}" sy="2.4" sz="${wall_h}"/>
-    <xacro:wall name="room_v_right_bot" x="1.8" y="-2.6" yaw="0" sx="${wall_t}" sy="2.8" sz="${wall_h}"/>
+    <!-- Vertikal vegg ved x = -0.8, med døråpning rundt y = 0 -->
+    <xacro:wall name="room_v_left_top" x="-0.8" y="1.0"  yaw="0" sx="${wall_t}" sy="1.5" sz="${wall_h}"/>
+    <xacro:wall name="room_v_left_bot" x="-0.8" y="-1.0" yaw="0" sx="${wall_t}" sy="1.5" sz="${wall_h}"/>
+    <!-- Vertikal vegg ved x = 0.9, med døråpning rundt y = -0.5 -->
+    <xacro:wall name="room_v_right_top" x="0.9" y="1.1"  yaw="0" sx="${wall_t}" sy="1.2" sz="${wall_h}"/>
+    <xacro:wall name="room_v_right_bot" x="0.9" y="-1.3" yaw="0" sx="${wall_t}" sy="1.4" sz="${wall_h}"/>
     <!-- Hindringer -->
     <!--
@@ -136,6 +140,6 @@
     -->
     <!-- Varme kilder -->
-    <xacro:thermal_box name="hot_target_1"  x="3.0"  y="1.0"  z="0.4" yaw="0"   sx="0.5" sy="0.5" sz="0.8" temp_k="360.0" r="1.0" g="0.2" b="0.2"/>
-    <xacro:thermal_box name="cold_target_1" x="-2.2" y="-1.4" z="0.4" yaw="0.3" sx="0.6" sy="0.4" sz="0.8" temp_k="285.0" r="0.2" g="0.4" b="1.0"/>
+    <xacro:thermal_box name="hot_target_1"  x="1.5"  y="0.5"  z="0.4" yaw="0"   sx="0.5" sy="0.5" sz="0.8" temp_k="360.0" r="1.0" g="0.2" b="0.2"/>
+    <xacro:thermal_box name="cold_target_1" x="-1.1" y="-0.8" z="0.4" yaw="0.3" sx="0.6" sy="0.4" sz="0.8" temp_k="285.0" r="0.2" g="0.4" b="1.0"/>
     <!-- Teddy Bear / Leketøy fra Gazebo Fuel -->
     <!--
